File: balun_eth_rj45/balun_eth_rj45.kicad_sch (KiCad schematic)
At the start: 17 parts, among them J1 RJE591885401 CAT6 NO-MAGNETICS, J2 SMA_A, J3 SMA_B, J4 SMA_C, J5 SMA_D, T1 ADT2-1T+, T2 ADT2-1T+, T3 ADT2-1T+, T4 ADT2-1T+

Commit message: feat: add complete VNA fixture design set
Parts:
- RCT1, RCT2, RCT3, RCT4: MPN 0 ohm 0805 -> 0805W8F0000T5E; Manufacturer ANY -> UNI-ROYAL
- RSH1: MPN (none) -> 0805W8F0000T5E; Manufacturer (none) -> UNI-ROYAL
- TP1, TP2: MPN (none) -> 5001; Manufacturer (none) -> Keystone Electronics
Connections:
- net GND: no longer RCT1.2, RCT2.2, RCT3.2, RCT4.2, T1.5, T2.5, T3.5, T4.5
- new net: RCT4.2, T4.5
- new net: RCT1.2, T1.5
- new net: RCT3.2, T3.5
- new net: RCT2.2, T2.5
Other:
- note added: "1. Passive DUT only. Disconnect PoE and all active Ethernet equipment before connecting the VNA."
- note added: "10. No TVS, common-mode choke, MagJack, series capacitors or on-board 50 ohm loads are added to the signal paths."
- note added: "1:2 impedance"
- note added: "2. Two identical PCB artworks; measure one path at a time and terminate all six unused SMA ports with 50 ohm loads."
- note added: "3. RCT1..RCT4 are DNP on this board. The default comparison condition is CT-FLOAT on both endpoint boards."
- note added: "4. CT-GND is a separate controlled comparison: fit all eight RCTs across two boards; do not mix CT states."
- note added: "5. This common CAD keeps RSH1 and CSH1 DNP. Final PCBA variants follow PCBA_PURCHASE_SCOPE_2026-09-03.md."
- note added: "50 ohm"
- note added: "6. RSH1 fitted = direct shield bond; CSH1 alone = optional AC bond; both DNP = floating. Never fit both together."
- note added: "7. Final shield variants are assembled by the supplier; legacy hand-fit property text is not a user soldering instruction."
- note added: "8. Coax O/S/L + THRU calibration leaves the PCB / balun response embedded. Keep REF/DUT fixture conditions fixed."
- note added: "9. Secondary convention P=pin 4, N=pin 6 is unchanged. Account for single-fixture polarity in phase/de-embedding work."
- note added: "A / RJ45 1(+) - 2(-)"
- note added: "ASSEMBLY / MEASUREMENT NOTES"
- note added: "B / RJ45 3(+) - 6(-)"
- note added: "C / RJ45 4(+) - 5(-)"
- note added: "Component pin numbers, not a mating-face drawing."
- note added: "D / RJ45 7(+) - 8(-)"
- note added: "DNP / CT FLOAT"
- note added: "DNP IN COMMON CAD"
- note added: "OPTIONAL AC BOND / DNP"
- note added: "PCBA: SHIELD-BONDED / SHIELD-FLOAT variants."
- note added: "RJ45 / FOUR-PAIR VNA FIXTURE"
- note added: "RJ45 / NO MAGNETICS"
- note added: "RJ45 이더넷 케이블 측정 지그 | 4-channel VNA fixture"
- note added: "SHIELD OPTIONS / TEST POINTS"
- note added: "Supplier fits RSH1 only on the BONDED boards."
- note removed: "CALIBRATION: coax SOLT at SMA cable ends; fixture remains embedded for Rev A A/B comparison"
- note removed: "CSH1 1nF/2kV (DNP)"
- note removed: "J1 FOOTPRINT VERIFIED: RJE59-188-5X01 Rev.C component-side hole pattern; mating face pin order 8..1"
- note removed: "J1 RJE591885401 CAT6 / SHIELDED / NO MAGNETICS"
- note removed: "J2 PAIR A / RJ45 1-2"
- note removed: "J3 PAIR B / RJ45 3-6"
- note removed: "J4 PAIR C / RJ45 4-5"
- note removed: "J5 PAIR D / RJ45 7-8"
- note removed: "No TVS, common-mode choke, MagJack, series capacitors, or onboard 50 ohm loads in the measurement path"
- note removed: "PAIR MAP: A=RJ45 1-2, B=3-6, C=4-5, D=7-8"
- note removed: "PASSIVE DUT ONLY - DO NOT CONNECT PoE OR ACTIVE ETHERNET"
- note removed: "RCT1 0R (DNP DEFAULT)"
- note removed: "RCT1..4: DNP default (CT-FLOAT); for CT-GND comparison fit all eight RCTs across both boards; no mixed states"
- note removed: "RCT2 0R (DNP DEFAULT)"
- note removed: "RCT3 0R (DNP DEFAULT)"
- note removed: "RCT4 0R (DNP DEFAULT)"
- note removed: "RSH1 0R (ASSEMBLY OPTION)"
- note removed: "SHIELD OPTIONS"
- note removed: "SHIELD: RSH1 fitted = direct; CSH1 alone = AC; both DNP = floating. Fit RSH1 on one board only; keep this state fixed across CT variants."
- note removed: "TP1 GND"
- note removed: "TP2 SHIELD"
- note removed: "UNUSED SMA PORTS: INSTALL EXTERNAL 50 ohm TERMINATORS (up to six for a two-board test)"
- title: 4-pair RJ45 VNA fixture, 50 ohm single-ended to 100 ohm differential -> RJ45 / FOUR-PAIR VNA FIXTURE
- moved on the sheet: T1, T2, T3, T4
