File: balun_slipring/m12_end/balun_slipring_m12.kicad_pcb (KiCad board)
At the start: 4 copper layers, 68 x 44 mm, 10 parts, among them J2 SMA_A, J3 SMA_B, T1 ADT2-1T+, T2 ADT2-1T+

Commit message: feat: finalize slip-ring fixtures and floating CT baseline
Parts:
- added J1: MB12FBAFF08ST-3 / VERIFY MECHANICS, balun_slipring_common:Finecables_MB12FBAFF08ST-3, B.Cu at (30.0, 42.0)
- RCT1, RCT2: moved to B.Cu
Connections:
- T1 pad 4: /PAIR_A_P_TBD -> /PAIR_TX_P
- T1 pad 6: /PAIR_A_N_TBD -> /PAIR_TX_N
- T2 pad 4: /PAIR_B_P_TBD -> /PAIR_RX_P
- T2 pad 6: /PAIR_B_N_TBD -> /PAIR_RX_N
Routing:
- net /PAIR_TX_N: track 0.00 -> 27.6 mm
- net /PAIR_TX_P: track 0.00 -> 27.6 mm
- net /PAIR_RX_N: track 0.00 -> 26.9 mm
- net /PAIR_RX_P: track 0.00 -> 26.9 mm
- net /GND: track 13.9 -> 25.0 mm
- net Net-(RCT2-Pad2): vias 0 -> 1
- net Net-(RCT1-Pad2): vias 0 -> 1
Other:
- board text added: "DOC MAP: TX / RX"
- board text added: "DRAFT 1 - DO NOT FAB"
- board text added: "M12 FEMALE / BACK SIDE CAND"
- board text added: "PIN 1 / A-KEY VERIFY"
- board text added: "PINS 5-8: NC"
- board text added: "RX"
- board text added: "SLIPRING M12 END / DOC MAP"
- board text added: "TX"
- board text added: "VERIFY MATING FACE / PANEL ACCESS"
- board text added: "VERIFY REV-504 CONTINUITY + J1 PIN 1 / KEY BEFORE FAB"
- board text removed: "A"
- board text removed: "B"
- board text removed: "DRAFT - DO NOT FAB"
- board text removed: "FOOTPRINT TBD"
- board text removed: "M12 AREA TBD"
- board text removed: "M12 FEMALE"
- board text removed: "MECHANICS TBD"
- board text removed: "NO ROUTING IN THIS GAP UNTIL CONTINUITY MAP IS VERIFIED"
- board text removed: "PINMAP TBD"
- board text removed: "SLIPRING M12 END / PINMAP TBD"

Commit message: feat: finalize JLC parts and measurement BOM
Parts:
- J2, J3: footprint Connector_Coaxial:SMA_Amphenol_132289_EdgeMount -> balun_slipring_common:SMA_MyAntenna_A-SMA-KE-16.5A_EdgeMount
- moved J2 0.30 mm to (85.8, 31.0)
- moved J3 0.30 mm to (85.8, 53.0)
Routing:
- net /GND: track 25.0 -> 46.4 mm

Commit message: feat: add complete VNA fixture design set
Routing:
- net /PAIR_RX_N: track 26.9 -> 27.6 mm
- net /PAIR_RX_P: track 26.9 -> 27.6 mm
Other:
- board text added: "M12 J1 / B-SIDE CAND"
- board text added: "슬립링 / SLIPRING"
- board text removed: "M12 FEMALE / BACK SIDE CAND"
- board text removed: "SLIPRING M12 END / DOC MAP"
