File: balun_slipring/molex_end/balun_slipring_molex.kicad_pcb (KiCad board)
At the start: 4 copper layers, 68 x 44 mm, 11 parts, among them J1 5055680471 / PINMAP TBD, J2 SMA_A, J3 SMA_B, T1 ADT2-1T+, T2 ADT2-1T+

Commit message: feat: finalize slip-ring fixtures and floating CT baseline
Parts:
- J1: value 5055680471 / PINMAP TBD -> 5055680571 / MATE FOR 5055650501; footprint balun_slipring_common:Molex_5055680471 -> balun_slipring_common:Molex_5055680571
- RCT1, RCT2: moved to B.Cu
Connections:
- J1 pad 1: /MOL_RAW1 -> /PAIR_TX_P
- J1 pad 2: /MOL_RAW2 -> /PAIR_TX_N
- J1 pad 3: /MOL_RAW3 -> /PAIR_RX_P
- J1 pad 4: /MOL_RAW4 -> /PAIR_RX_N
- T1 pad 4: /PAIR_A_P_TBD -> /PAIR_TX_P
- T1 pad 6: /PAIR_A_N_TBD -> /PAIR_TX_N
- T2 pad 4: /PAIR_B_P_TBD -> /PAIR_RX_P
- T2 pad 6: /PAIR_B_N_TBD -> /PAIR_RX_N
Routing:
- net /PAIR_RX_N: track 0.00 -> 31.9 mm
- net /PAIR_RX_P: track 0.00 -> 31.9 mm
- net /PAIR_TX_N: track 0.00 -> 31.1 mm
- net /PAIR_TX_P: track 0.00 -> 31.1 mm
- net /GND: track 13.9 -> 25.0 mm
- net Net-(RCT2-Pad2): vias 0 -> 1
- net Net-(RCT1-Pad2): vias 0 -> 1
Other:
- board text added: "5055680571 CAND"
- board text added: "DOC MAP: TX / RX"
- board text added: "DRAFT 1 - DO NOT FAB"
- board text added: "RX"
- board text added: "SLIPRING MOLEX END / DOC MAP"
- board text added: "TX"
- board text added: "VERIFY REV-504 CONTINUITY + J1 PIN 1 / KEY BEFORE FAB"
- board text removed: "5055680471"
- board text removed: "A"
- board text removed: "B"
- board text removed: "DRAFT - DO NOT FAB"
- board text removed: "NO ROUTING IN THIS GAP UNTIL CONTINUITY MAP IS VERIFIED"
- board text removed: "PINMAP TBD"
- board text removed: "SLIPRING MOLEX END / PINMAP TBD"

Commit message: feat: finalize JLC parts and measurement BOM
Parts:
- J2, J3: footprint Connector_Coaxial:SMA_Amphenol_132289_EdgeMount -> balun_slipring_common:SMA_MyAntenna_A-SMA-KE-16.5A_EdgeMount
- moved J2 0.30 mm to (85.8, 31.0)
- moved J3 0.30 mm to (85.8, 53.0)
Routing:
- net /GND: track 25.0 -> 46.4 mm

Commit message: feat: add complete VNA fixture design set
Parts:
- J1: value 5055680571 / MATE FOR 5055650501 -> 5055680571 / 505565 SERIES MATE CAND
