File: adapters/m12_llc/m12_llc.kicad_pcb (KiCad board)
At the start: 4 copper layers, 66 x 40 mm, 7 parts, among them J1 RJ45 RJE591885401, J2 MB12MBAFF08ST-3

Commit message: Verify JLC stack impedance, update PCB widths, and document ordering options with screenshots
Other:
- board text added: "A-DRAFT / VERIFY MATE + CAM"
- board text removed: "A-DRAFT / VERIFY MATE + IMPEDANCE"
Changed lines of the file:
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@@
 		(rev "A-DRAFT")
 		(comment 1 "M12 MALE / LLC; 1,5,6,7 NC; VERIFY MATE")
-		(comment 2 "JLC04161H-7628 / 100R trunk W0.23 G0.22 / verify manufacturer mating")
+		(comment 2 "JLC04161H-7628 / 100R trunk W0.234 G0.216 / verify manufacturer mating")
 	)
 	(layers
@@
 		(layer "Edge.Cuts")
 	)
-	(gr_text "A-DRAFT / VERIFY MATE + IMPEDANCE"
+	(gr_text "A-DRAFT / VERIFY MATE + CAM"
 		(at 33 37 0)
 		(layer "F.SilkS")
@@
 		(start 26 22.209712)
 		(end 30 15)
-		(width 0.23)
+		(width 0.234)
 		(layer "F.Cu")
 		(net "/PAIR_A_N")
@@
 		(start 22 17.41)
 		(end 26 22.209712)
-		(width 0.23)
+		(width 0.234)
 		(layer "F.Cu")
 		(net "/PAIR_A_N")
@@
 		(start 30 15)
 		(end 41 15)
-		(width 0.23)
+		(width 0.234)
 		(layer "F.Cu")
 		(net "/PAIR_A_N")
@@
 		(start 41 15)
 		(end 46.502243 15)
-		(width 0.23)
+		(width 0.234)
 		(layer "F.Cu")
 		(net "/PAIR_A_N")
@@
 		(start 46.502243 15)
 		(end 46.502243 17.693656)
-		(width 0.23)
+		(width 0.234)
 		(layer "F.Cu")
 		(net "/PAIR_A_N")
@@
 		(start 30 20)
 		(end 42 20)
-		(width 0.23)
+		(width 0.234)
 		(layer "B.Cu")
 		(net "/PAIR_B_P")
@@
 		(start 43.5 19.5)
 		(end 45.276763 19.617274)
-		(width 0.23)
+		(width 0.234)
 		(layer "B.Cu")
 		(net "/PAIR_B_P")
@@
 		(start 42 20)
 		(end 43.5 19.5)
-		(width 0.23)
+		(width 0.234)
 		(layer "B.Cu")
 		(net "/PAIR_B_P")
@@
 		(start 26 19.215)
 		(end 30 20)
-		(width 0.23)
+		(width 0.234)
 		(layer "B.Cu")
 		(net "/PAIR_B_P")
@@
 		(start 22 18.43)
 		(end 26 19.215)
-		(width 0.23)
+		(width 0.234)
 		(layer "B.Cu")
 		(net "/PAIR_B_P")
@@
 		(start 22 21.49)
 		(end 26 22.452602)
-		(width 0.23)
+		(width 0.234)
 		(layer "B.Cu")
 		(net "/PAIR_B_N")
@@
 		(start 43.5 22.4)
 		(end 45.924549 21.804162)
-		(width 0.23)
+		(width 0.234)
 		(layer "B.Cu")
 		(net "/PAIR_B_N")
@@
 		(start 30 20.45)
 		(end 42 20.45)
-		(width 0.23)
+		(width 0.234)
 		(layer "B.Cu")
 		(net "/PAIR_B_N")
@@
 		(start 42 20.45)
 		(end 43.5 22.4)
-		(width 0.23)
+		(width 0.234)
 		(layer "B.Cu")
 		(net "/PAIR_B_N")
@@
 		(start 26 22.452602)
 		(end 30 20.45)
-		(width 0.23)
+		(width 0.234)
 		(layer "B.Cu")
 		(net "/PAIR_B_N")
@@
 		(start 41 14.55)
 		(end 48 14.55)
-		(width 0.23)
+		(width 0.234)
 		(layer "F.Cu")
 		(net "/PAIR_A_P")
@@
 		(start 22 16.39)
 		(end 26 15.47)
-		(width 0.23)
+		(width 0.234)
 		(layer "F.Cu")
 		(net "/PAIR_A_P")
@@
 		(start 26 15.47)
 		(end 30 14.55)
-		(width 0.23)
+		(width 0.234)
 		(layer "F.Cu")
 		(net "/PAIR_A_P")
@@
 		(start 30 14.55)
 		(end 41 14.55)
-		(width 0.23)
+		(width 0.234)
 		(layer "F.Cu")
 		(net "/PAIR_A_P")
@@
 		(start 48 14.55)
 		(end 48 20)
-		(width 0.23)
+		(width 0.234)
 		(layer "F.Cu")
 		(net "/PAIR_A_P")
