File: adapters/m12_slipring/m12_slipring.kicad_pcb (KiCad board)
At the start: 4 copper layers, 66 x 40 mm, 7 parts, among them J1 RJ45 RJE591885401, J2 MB12FBAFF08ST-3

Commit message: Verify JLC stack impedance, update PCB widths, and document ordering options with screenshots
Other:
- board text added: "A-DRAFT / VERIFY MATE + CAM"
- board text removed: "A-DRAFT / VERIFY MATE + IMPEDANCE"
Changed lines of the file:
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@@
 		(rev "A-DRAFT")
 		(comment 1 "M12 FEMALE / SLIPRING; 5-8 NC; VERIFY MATE")
-		(comment 2 "JLC04161H-7628 / 100R trunk W0.23 G0.22 / verify manufacturer mating")
+		(comment 2 "JLC04161H-7628 / 100R trunk W0.234 G0.216 / verify manufacturer mating")
 	)
 	(layers
@@
 		(layer "Edge.Cuts")
 	)
-	(gr_text "A-DRAFT / VERIFY MATE + IMPEDANCE"
+	(gr_text "A-DRAFT / VERIFY MATE + CAM"
 		(at 33 37 0)
 		(layer "F.SilkS")
@@
 		(start 22 16.39)
 		(end 26 16.795)
-		(width 0.23)
+		(width 0.234)
 		(layer "F.Cu")
 		(net "/PAIR_A_P")
@@
 		(start 42 17.2)
 		(end 44 17.2)
-		(width 0.23)
+		(width 0.234)
 		(layer "F.Cu")
 		(net "/PAIR_A_P")
@@
 		(start 26 16.795)
 		(end 30 17.2)
-		(width 0.23)
+		(width 0.234)
 		(layer "F.Cu")
 		(net "/PAIR_A_P")
@@
 		(start 44 17.2)
 		(end 45.924549 18.195838)
-		(width 0.23)
+		(width 0.234)
 		(layer "F.Cu")
 		(net "/PAIR_A_P")
@@
 		(start 30 17.2)
 		(end 42 17.2)
-		(width 0.23)
+		(width 0.234)
 		(layer "F.Cu")
 		(net "/PAIR_A_P")
@@
 		(start 30 17.65)
 		(end 42 17.65)
-		(width 0.23)
+		(width 0.234)
 		(layer "F.Cu")
 		(net "/PAIR_A_N")
@@
 		(start 26 20.311796)
 		(end 30 17.65)
-		(width 0.23)
+		(width 0.234)
 		(layer "F.Cu")
 		(net "/PAIR_A_N")
@@
 		(start 43.5 19.8)
 		(end 45.276763 20.382726)
-		(width 0.23)
+		(width 0.234)
 		(layer "F.Cu")
 		(net "/PAIR_A_N")
@@
 		(start 42 17.65)
 		(end 43.5 19.8)
-		(width 0.23)
+		(width 0.234)
 		(layer "F.Cu")
 		(net "/PAIR_A_N")
@@
 		(start 22 17.41)
 		(end 26 20.311796)
-		(width 0.23)
+		(width 0.234)
 		(layer "F.Cu")
 		(net "/PAIR_A_N")
@@
 	(segment
 		(start 30 22.7)
-		(end 42 22.7)
-		(width 0.23)
+		(end 42.05 22.7)
+		(width 0.234)
 		(layer "B.Cu")
 		(net "/PAIR_B_P")
 	)
 	(segment
-		(start 42 22.7)
+		(start 42.05 22.7)
 		(end 46.502243 24)
-		(width 0.23)
+		(width 0.234)
 		(layer "B.Cu")
 		(net "/PAIR_B_P")
@@
 		(start 22 18.43)
 		(end 26 18.518824)
-		(width 0.23)
+		(width 0.234)
 		(layer "B.Cu")
 		(net "/PAIR_B_P")
@@
 		(start 26 18.518824)
 		(end 30 22.7)
-		(width 0.23)
+		(width 0.234)
 		(layer "B.Cu")
 		(net "/PAIR_B_P")
@@
 		(start 46.502243 24)
 		(end 46.502243 22.306344)
-		(width 0.23)
+		(width 0.234)
 		(layer "B.Cu")
 		(net "/PAIR_B_P")
@@
 		(start 42 23.15)
 		(end 44 24.45)
-		(width 0.23)
+		(width 0.234)
 		(layer "B.Cu")
 		(net "/PAIR_B_N")
@@
 		(start 49.497757 24.45)
 		(end 49.497757 22.306344)
-		(width 0.23)
+		(width 0.234)
 		(layer "B.Cu")
 		(net "/PAIR_B_N")
@@
 		(start 22 21.49)
 		(end 26 22.32)
-		(width 0.23)
+		(width 0.234)
 		(layer "B.Cu")
 		(net "/PAIR_B_N")
@@
 		(start 44 24.45)
 		(end 49.497757 24.45)
-		(width 0.23)
+		(width 0.234)
 		(layer "B.Cu")
 		(net "/PAIR_B_N")
@@
 		(start 30 23.15)
 		(end 42 23.15)
-		(width 0.23)
+		(width 0.234)
 		(layer "B.Cu")
 		(net "/PAIR_B_N")
@@
 		(start 26 22.32)
 		(end 30 23.15)
-		(width 0.23)
+		(width 0.234)
 		(layer "B.Cu")
 		(net "/PAIR_B_N")

Commit message: Review M12 slipring routing and enforce pair constraints
Parts:
- moved TP1 2.39 mm to (37.1, 29.1)
- turned J2 to -30 degrees
Routing:
- net /PAIR_A_P: track 29.2 -> 32.8 mm
- net /PAIR_A_N: track 29.2 -> 31.9 mm
- net /PAIR_B_P: track 33.2 -> 32.3 mm
- net /SHIELD: vias 10 -> 8
